Commit message: Updated

File: ar_bot_description/urdf/ar_bot.xacro (robot description, xacro)
@@ -13,4 +13,7 @@
     <material name="blue">
         <color rgba="0 0 0.8 1" />
+    </material>
+    <material name="neon_blue">
+        <color rgba="0 100 255 1" />
     </material>
     <material name="black">
