Commit message: Fixed cache performance structure

File: ar_bot_description/urdf/ar_bot.urdf (robot description, URDF)
Before this commit: robot visual, 4 links, 3 joints
Links:
- link base_link: mass None -> 0.028

Commit message: clean up

File: ar_bot_description/urdf/ar_bot.urdf (robot description, URDF)
Before this commit: robot arbot, 4 links, 3 joints
Links:
- link base_link: mass 0.028 -> 0.05
- link caster_wheel: mass None -> 0.01
- link left_wheel: mass None -> 0.01
- link right_wheel: mass None -> 0.01

File: ar_bot_description/urdf/ar_bot.xacro (robot description, xacro)
@@ -33,5 +33,7 @@
             </geometry>
         </collision>
-        <xacro:solid_cuboid_inertia mass="0.028" height="0.08" depth="0.082" width="0.078"/>
+        <xacro:solid_cuboid_inertia mass="0.05" height="0.08" depth="0.082" width="0.078">
+            <origin rpy="0 0 0.03" xyz="0 0 0" />
+        </xacro:solid_cuboid_inertia>
     </link>
     <joint name="right_wheel_joint" type="continuous">
@@ -53,4 +55,7 @@
             </geometry>
         </collision>
+        <xacro:solid_cylinder_inertia mass="0.01" height="0.008" radius="0.03">
+            <origin rpy="0 0 0" xyz="0 0 0" />
+        </xacro:solid_cylinder_inertia>
     </link>
     <joint name="left_wheel_joint" type="continuous">
@@ -72,4 +77,7 @@
             </geometry>
         </collision>
+        <xacro:solid_cylinder_inertia mass="0.01 " height="0.008" radius="0.03">
+            <origin rpy="0 0 0" xyz="0 0 0" />
+        </xacro:solid_cylinder_inertia>
     </link>
     <joint name="caster_wheel_joint" type="fixed">
@@ -90,4 +98,7 @@
             </geometry>
         </collision>
+        <xacro:solid_sphere_inertia mass="0.01" radius="0.006">
+            <origin rpy="0 0 0" xyz="0 0 0" />
+        </xacro:solid_sphere_inertia>
     </link>
 </robot>

File: ar_bot_description/urdf/inertial_macros.xacro (robot description, xacro)
@@ -1,9 +1,15 @@
 <?xml version="1.0"?>
+<!--
+Purpose:
+    xacro interia calculation macro
+Based off of:
+    - the ROS URDF Tutorial: https://github.com/ros/urdf_tutorial/blob/master/urdf/06-flexible.urdf
+    - URDF Tutorial by Articulated Robotics:
+        https://github.com/joshnewans/articubot_one/blob/d5aa5e9bc9039073c0d8fd7fe426e170be79c087/description/robot_core.xacro
+-->
 <robot xmlns:xacro="http://www.ros.org/wiki/xacro">
-    <!-- Specify some standard inertial calculations
-    https://en.wikipedia.org/wiki/List_of_moments_of_inertia -->
-    <!-- These make use of xacro's mathematical functionality -->
-    <xacro:macro name="solid_sphere_inertia" params="mass radius">
+    <xacro:macro name="solid_sphere_inertia" params="mass radius *origin">
         <inertial>
+            <xacro:insert_block name="origin"/>
             <mass value="${mass}" />
             <inertia ixx="${(2/5) * mass * (radius*radius)}" ixy="0.0" ixz="0.0"
@@ -12,6 +18,7 @@
         </inertial>
     </xacro:macro>
-    <xacro:macro name="solid_cuboid_inertia" params="mass height depth width">
+    <xacro:macro name="solid_cuboid_inertia" params="mass height depth width *origin">
         <inertial>
+            <xacro:insert_block name="origin"/>
             <mass value="${mass}" />
             <inertia ixx="${(mass*(height*height+depth*depth))/12}" ixy="0" ixz="0"
@@ -21,6 +28,7 @@
         </inertial>
     </xacro:macro>
-    <xacro:macro name="solid_cylinder_inertia" params="mass height radius">
+    <xacro:macro name="solid_cylinder_inertia" params="mass height radius *origin">
         <inertial>
+            <xacro:insert_block name="origin"/>
             <mass value="${mass}" />
             <inertia ixx="${(1/12) * mass * (3*radius*radius + height*height)}" ixy="0.0" ixz="0.0"
